File: hardware/motor-driver/motor-driver.kicad_sch (KiCad schematic)
At the start: 23 parts, among them J1 Screw_Terminal_01x02, J10 Conn_01x02, J11 Conn_01x02, J12 Conn_01x02, J2 Screw_Terminal_01x02, J3 Screw_Terminal_01x02, J4 Conn_01x06, J5 Conn_01x06, J6 Conn_01x04, J7 Conn_01x04, J8 Conn_01x04, J9 Conn_01x04, Q1 AO4407A, U1 TLE9201SG, U2 TLE9201SG, U3 RP2040-castaway

Commit message: Initial commit for  version 2
Parts:
- removed U3: RP2040-castaway, shurik-personal:RP2040-castaway, symbol shurik-personal:RP2040-castaway
- added C10, C11, C12, C13, C14, C15, C16, C17, C18, C23, C9: 100nF, Capacitor_SMD:C_0402_1005Metric, symbol Device:C
- added C19: 220nF, Capacitor_SMD:C_0402_1005Metric, symbol Device:C
- added C2, C22, C3: 10uF, Capacitor_SMD:C_0805_2012Metric, symbol Device:C
- added C20, C21: 30pF, Capacitor_SMD:C_0402_1005Metric, symbol Device:C
- added C4: 10uF, Capacitor_SMD:C_1206_3216Metric, symbol Device:C
- added C5, C6: 1uF, Capacitor_SMD:C_0402_1005Metric, symbol Device:C
- added D2: B5819W, Diode_SMD:D_SOD-123, symbol Device:D_Schottky
- added D3, D4: WS2812B-mini, LED_SMD:LED_SK6812MINI_PLCC4_3.5x3.5mm_P1.75mm, symbol shurik-personal:WS2812B-mini
- added D5: MM1Z12, Diode_SMD:D_SOD-123, symbol Device:D_Zener
- added D6: SMF22CA, Diode_SMD:D_SOD-123F, symbol Device:D_TVS
- added J13: Conn_01x01, Connector_PinHeader_2.54mm:PinHeader_1x01_P2.54mm_Vertical, symbol Connector_Generic:Conn_01x01
- added J14: USB_B_Micro, shurik-personal:USB_Micro-B_Amphenol_10118194_Horizontal, symbol Connector:USB_B_Micro
- added JP3: SolderJumper_2_Open, Jumper:SolderJumper-2_P1.3mm_Open_TrianglePad1.0x1.5mm, symbol Jumper:SolderJumper_2_Open
- added L1: 10uH, Inductor_SMD:L_Taiyo-Yuden_NR-40xx, symbol Device:L_Small
- added R10, R8, R9: 10k, Resistor_SMD:R_0402_1005Metric, symbol Device:R_Small
- added R11, R12: 54.9k, Resistor_SMD:R_0402_1005Metric, symbol Device:R_Small
- added R2, R4: 1k, Resistor_SMD:R_0402_1005Metric, symbol Device:R
- added R3: 10K, Resistor_SMD:R_0402_1005Metric, symbol Device:R
- added R5, R6: 27, Resistor_SMD:R_0402_1005Metric, symbol Device:R
- added R7: 10k, Resistor_SMD:R_0402_1005Metric, symbol Device:R
- added SW1: SW_Push, Button_Switch_SMD:SW_SPST_PTS810, symbol Switch:SW_Push
- added U3: LM2842X, Package_TO_SOT_SMD:TSOT-23-6, symbol Regulator_Switching:LM2842X
- added U4: AP2120N-3.3, Package_TO_SOT_SMD:SOT-23, symbol Regulator_Linear:AP2127N-3.3
- added U5: RP2040, RP2040_minimal:RP2040-QFN-56, symbol MCU_RaspberryPi_RP2040:RP2040
- added U6: W25Q16JVS, Package_SO:SOIC-8_5.23x5.23mm_P1.27mm, symbol Memory_Flash:W25Q128JVS
- added Y1: X322512MSB4SI, Crystal:Crystal_SMD_Abracon_ABM8G-4Pin_3.2x2.5mm, symbol Device:Crystal_GND24
- C7: renamed from C2; footprint Capacitor_SMD:C_0805_2012Metric -> Capacitor_SMD:C_0402_1005Metric; LCSC (none) -> C1525
- C8: renamed from C3; footprint Capacitor_SMD:C_0805_2012Metric -> Capacitor_SMD:C_0402_1005Metric; LCSC (none) -> C1525
- D1: footprint LED_SMD:LED_0805_2012Metric -> LED_SMD:LED_0603_1608Metric; LCSC (none) -> C72043
- J1, J2, J3: footprint TerminalBlock_Phoenix:TerminalBlock_Phoenix_MKDS-1,5-2_1x02_P5.00mm_Horizontal -> shurik-personal:TerminalBlock_Phoenix_MKDS-1,5-2_1x02_P5.00mm_Horizontal_nosilk
- J10, J11: footprint shurik-personal:JST_VH_S2P-VH_1x02_P3.96mm_Horizontal -> Shurik:JST_VH_B2P-VH-B_1x02_P3.96mm_Vertical-nosilk
- J12: footprint shurik-personal:JST_VH_S2P-VH_1x02_P3.96mm_Horizontal -> Connector_AMASS:AMASS_XT30UPB-M_1x02_P5.0mm_Vertical
- J6, J7: LCSC (none) -> C239522
- Q1: value AO4407A -> AO4407C; LCSC (none) -> C469397
- R1: value 2K -> 3.3k; footprint Resistor_SMD:R_0805_2012Metric -> Resistor_SMD:R_0402_1005Metric; LCSC (none) -> C25890
- U1, U2: LCSC (none) -> C2653438
Connections:
- net +3V3: now also C11.1, C12.1, C13.1, C14.1, C15.1, C16.1, C17.1, C18.1, C2.1, C23.1, C6.1, D3.1 (VDD), D4.1 (VDD), R10.1, R3.1, R7.1, R9.1, U4.2 (VO), U5.1 (IOVDD), U5.10 (IOVDD), U5.22 (IOVDD), U5.33 (IOVDD), U5.42 (IOVDD), U5.43 (ADC_AVDD), U5.44 (VREG_IN), U5.48 (USB_VDD), U5.49 (IOVDD), U6.8 (VCC); no longer J6.2 (Pin_2), J7.2 (Pin_2)
- net ENC1_A: now also U5.30 (GPIO19)
- net ENC1_B: now also U5.29 (GPIO18)
- net ENC2_A: now also U5.9 (GPIO7)
- net ENC2_B: now also U5.8 (GPIO6)
- net GND: now also C10.2, C11.2, C12.2, C13.2, C14.2, C15.2, C16.2, C17.2, C18.2, C2.2, C20.2, C21.2, C22.1, C23.2, C3.1, C4.1, C5.2, C6.2, C9.2, D2.2 (A), D3.3 (VSS), D4.3 (VSS), D6.1 (A1), J14.5 (GND), J14.6 (Shield), JP3.2 (B), R12.2, R8.2, SW1.1, U3.2 (GND), U4.1 (GND), U5.19 (TESTEN), U5.57 (GND), U6.4 (GND), Y1.2, Y1.4; no longer Q1.4 (G)
- net M1A: now also J10.2 (Pin_2); no longer J10.1 (Pin_1)
- net M1B: now also J10.1 (Pin_1); no longer J10.2 (Pin_2)
- net M1_DIR: now also U5.31 (GPIO20)
- net M1_FLAG: now also U5.36 (GPIO24)
- net M1_PWM: now also U5.40 (GPIO28_ADC2)
- net M2A: now also J11.2 (Pin_2); no longer J11.1 (Pin_1)
- net M2B: now also J11.1 (Pin_1); no longer J11.2 (Pin_2)
- net M2_DIR: now also U5.4 (GPIO2)
- net M2_FLAG: now also U5.7 (GPIO5)
- net M2_PWM: now also U5.13 (GPIO10)
- net SCL: now also R9.2, U5.3 (GPIO1)
- net SDA: now also R10.2, U5.2 (GPIO0)
- net VBUS: now also D6.2 (A2)
- net VCC: now also C4.2, D5.1 (K), U3.4 (EN), U3.5 (VIN); no longer D1.2 (A)
- net ADDR_0: now reaches JP1.1 (A)
- net ADDR_0: now also U5.15 (GPIO12)
- net ADDR_1: now reaches JP2.1 (A)
- net ADDR_1: now also U5.16 (GPIO13)
- net ENABLE renamed M1_ENABLE
- net M1_ENABLE: now also U5.39 (GPIO27_ADC1); no longer U2.11 (DIS)
- new net: C20.1, R4.2, Y1.1
- new net: R11.2, R8.1, U3.3 (FB)
- new net: C19.1, U3.1 (BOOST)
- new net: C19.2, D2.1 (K), L1.1, U3.6 (SW)
- new net: R6.2, U5.46 (USB_DM)
- new net: D3.4 (DIN), D4.2 (DOUT)
- new net: D5.2 (A), Q1.4 (G), R12.1
- new net: R5.2, U5.47 (USB_DP)
- new net +1V1: C10.1, C5.1, C9.1, U5.23 (DVDD), U5.45 (VREG_VOUT), U5.50 (DVDD)
- new net +5V: C22.2, C3.2, D1.2 (A), J14.1 (VBUS), L1.2, R11.1, U4.3 (VI)
- new net ADDR_2: JP3.1 (A), U5.17 (GPIO14)
- new net M2_ENABLE: U2.11 (DIS), U5.14 (GPIO11)
- new net NEOPIXEL: D4.4 (DIN), U5.5 (GPIO3)
- new net QSPI_SCLK: U5.52 (QSPI_SCLK), U6.6 (CLK)
- new net QSPI_SD0: U5.53 (QSPI_SD0), U6.5 (DI(IO0))
- new net QSPI_SD1: U5.55 (QSPI_SD1), U6.2 (DO(IO1))
- new net QSPI_SD2: U5.54 (QSPI_SD2), U6.3 (IO2)
- new net QSPI_SD3: U5.51 (QSPI_SD3), U6.7 (IO3)
- new net QSPI_SS: R2.1, R3.2, U5.56 (QSPI_SS), U6.1 (~{CS})
- new net RUN: R7.2, SW1.2, U5.26 (RUN)
- new net USB_D+: J14.3 (D+), R5.1
- new net USB_D-: J14.2 (D-), R6.1
- new net XIN: C21.1, U5.20 (XIN), Y1.3
- new net XOUT: R4.1, U5.21 (XOUT)
- new net ~{USB_BOOT}: J13.1 (Pin_1), R2.2
- no-connect marks 0 -> 14
Other:
- note added: "C1, C4 must be rated for 35V or more"
- note added: "Crystal"
- note added: "Flash"
- note added: "I2C connectors"
- note added: "Make sure C5 is close to pin 45 of RP2040"
- note added: "Make sure C6 is close to pin 44 of RP2040"
- note added: "Make sure R5 and R6 are close to RP2040"
- note added: "Motor drivers"
- note added: "Neopixels"
- note added: "Pin 2 is I2C 3.3v - unconnected"
- note added: "Power"
- moved on the sheet: C1, C7, C8, D1, J1, J10, J11, J2, J4, J5, J6, J7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
