File: hardware/motor-driver/motor-driver.kicad_sch (KiCad schematic)
At the start: 75 parts, among them J1 Screw_Terminal_01x02, J10 Conn_01x02, J11 Conn_01x02, J12 Conn_01x02, J13 Conn_01x01, J14 USB_B_Micro, J2 Screw_Terminal_01x02, J3 Screw_Terminal_01x02, J4 Conn_01x06, J5 Conn_01x06, J6 Conn_01x04, J7 Conn_01x04, J8 Conn_01x04, J9 Conn_01x04, Q1 AO4407C, SW1 SW_Push, U1 DRV8874PWPR, U2 DRV8874PWPR, U3 LM2842X, U4 AP2112K-3.3, U5 RP2040, U6 W25Q16JVS, U7 74LVC1G126, Y1 X322512MSB4SI

Commit message: version 3.0.0-beta1
Parts:
- L1: footprint Inductor_SMD:L_Taiyo-Yuden_NR-40xx -> Inductor_SMD:L_Sunlord_SWPA4018S; LCSC C36405 -> C83442
Connections:
- net M1_DIR: now also U5.37 (GPIO25); no longer U5.39 (GPIO27_ADC1)
- net M1_ENABLE: now also U5.36 (GPIO24); no longer U5.38 (GPIO26_ADC0)
- net M1_PWM: now also U5.38 (GPIO26_ADC0); no longer U5.40 (GPIO28_ADC2)
- net M1_SENSE: now also U5.39 (GPIO27_ADC1)
- net M2_SENSE: now also U5.40 (GPIO28_ADC2)
- net at JP4.2 (B): now also U5.34 (GPIO22); no longer U5.36 (GPIO24)
- net at JP3.2 (B): now also U5.35 (GPIO23); no longer U5.37 (GPIO25)
- no-connect marks 11 -> 9
Changed lines of the file:
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@@
   (no_connect (at 323.85 127))
   (no_connect (at 323.85 139.7))
-  (no_connect (at 323.85 142.24))
-  (no_connect (at 323.85 144.78))
   (no_connect (at 260.35 151.13))
   (no_connect (at 260.35 153.67))
@@
     (stroke (width 0) (type default))
   )
+  (wire (pts (xy 323.85 142.24) (xy 356.87 142.24))
+    (stroke (width 0) (type default))
+  )
   (wire (pts (xy 387.35 73.66) (xy 396.24 73.66))
     (stroke (width 0) (type default))
@@
     (stroke (width 0) (type default))
   )
-  (wire (pts (xy 356.87 147.32) (xy 356.87 151.13))
+  (wire (pts (xy 356.87 142.24) (xy 356.87 151.13))
     (stroke (width 0) (type default))
   )
@@
     (stroke (width 0) (type default))
   )
+  (wire (pts (xy 323.85 144.78) (xy 349.25 144.78))
+    (stroke (width 0) (type default))
+  )
   (wire (pts (xy 63.5 60.96) (xy 72.39 60.96))
     (stroke (width 0) (type default))
@@
     (stroke (width 0) (type default))
   )
+  (wire (pts (xy 323.85 149.86) (xy 339.09 149.86))
+    (stroke (width 0) (type default))
+  )
   (wire (pts (xy 271.78 34.29) (xy 271.78 35.56))
     (stroke (width 0) (type default))
@@
     (stroke (width 0) (type default))
   )
-  (wire (pts (xy 323.85 149.86) (xy 349.25 149.86))
-    (stroke (width 0) (type default))
-  )
   (wire (pts (xy 66.04 20.32) (xy 76.2 20.32))
     (stroke (width 0) (type default))
@@
     (stroke (width 0) (type default))
   )
+  (wire (pts (xy 323.85 147.32) (xy 339.09 147.32))
+    (stroke (width 0) (type default))
+  )
   (wire (pts (xy 320.04 213.36) (xy 326.39 213.36))
     (stroke (width 0) (type default))
@@
     (stroke (width 0) (type solid))
   )
-  (wire (pts (xy 323.85 147.32) (xy 356.87 147.32))
-    (stroke (width 0) (type default))
-  )
   (wire (pts (xy 49.53 30.48) (xy 49.53 33.02))
     (stroke (width 0) (type default))
@@
     (stroke (width 0) (type default))
   )
-  (wire (pts (xy 349.25 149.86) (xy 349.25 151.13))
+  (wire (pts (xy 349.25 144.78) (xy 349.25 151.13))
     (stroke (width 0) (type default))
   )
@@
     (effects (font (size 1.27 1.27)) (justify left bottom))
   )
-  (label "M1_DIR" (at 339.09 157.48 180) (fields_autoplaced)
-    (effects (font (size 1.27 1.27)) (justify right bottom))
-  )
   (label "ENC1_A" (at 129.54 219.71 0) (fields_autoplaced)
     (effects (font (size 1.27 1.27)) (justify left bottom))
   )
+  (label "M1_PWM" (at 339.09 154.94 180) (fields_autoplaced)
+    (effects (font (size 1.27 1.27)) (justify right bottom))
+  )
   (label "VREF" (at 198.12 250.19 0) (fields_autoplaced)
     (effects (font (size 1.27 1.27)) (justify left bottom))
@@
     (effects (font (size 1.27 1.27)) (justify left bottom))
   )
+  (label "M1_SENSE" (at 339.09 157.48 180) (fields_autoplaced)
+    (effects (font (size 1.27 1.27)) (justify right bottom))
+  )
   (label "M2B" (at 273.05 220.98 0) (fields_autoplaced)
     (effects (font (size 1.27 1.27)) (justify left bottom))
@@
     (effects (font (size 1.27 1.27)) (justify right bottom))
   )
+  (label "M1_DIR" (at 339.09 149.86 180) (fields_autoplaced)
+    (effects (font (size 1.27 1.27)) (justify right bottom))
+  )
   (label "ADDR_2" (at 339.09 121.92 180) (fields_autoplaced)
     (effects (font (size 1.27 1.27)) (justify right bottom))
   )
+  (label "M1_ENABLE" (at 339.09 147.32 180) (fields_autoplaced)
+    (effects (font (size 1.27 1.27)) (justify right bottom))
+  )
   (label "QSPI_SD1" (at 246.38 93.98 0) (fields_autoplaced)
     (effects (font (size 1.27 1.27)) (justify left bottom))
@@
     (effects (font (size 1.27 1.27)) (justify right bottom))
   )
-  (label "M1_ENABLE" (at 339.09 154.94 180) (fields_autoplaced)
-    (effects (font (size 1.27 1.27)) (justify right bottom))
-  )
   (label "QSPI_SD2" (at 215.9 52.07 180) (fields_autoplaced)
     (effects (font (size 1.27 1.27)) (justify right bottom))
@@
     (effects (font (size 1.27 1.27)) (justify right bottom))
   )
-  (label "M1_PWM" (at 339.09 160.02 180) (fields_autoplaced)
-    (effects (font (size 1.27 1.27)) (justify right bottom))
-  )
   (label "TX" (at 19.05 120.65 0) (fields_autoplaced)
     (effects (font (size 1.27 1.27)) (justify left bottom))
@@
     (effects (font (size 1.27 1.27)) (justify left bottom))
   )
+  (label "M2_SENSE" (at 339.09 160.02 180) (fields_autoplaced)
+    (effects (font (size 1.27 1.27)) (justify right bottom))
+  )
   (label "ENC2_B" (at 339.09 101.6 180) (fields_autoplaced)
     (effects (font (size 1.27 1.27)) (justify right bottom))
@@
       (effects (font (size 1.27 1.27)))
     )
-    (property "Footprint" "Inductor_SMD:L_Taiyo-Yuden_NR-40xx" (at 52.07 60.96 0)
+    (property "Footprint" "Inductor_SMD:L_Sunlord_SWPA4018S" (at 52.07 60.96 0)
       (effects (font (size 1.27 1.27)) hide)
     )
-    (property "Datasheet" "~" (at 52.07 60.96 0)
+    (property "Datasheet" "https://www.lcsc.com/datasheet/lcsc_datasheet_2310251551_Sunlord-SWPA4018S100MT_C83442.pdf" (at 52.07 60.96 0)
       (effects (font (size 1.27 1.27)) hide)
     )
-    (property "LCSC" "C36405" (at 52.07 60.96 0)
+    (property "LCSC" "C83442" (at 52.07 60.96 0)
       (effects (font (size 1.27 1.27)) hide)
     )
@@
       (effects (font (size 1.27 1.27)) hide)
     )
-    (property "Datasheet" "~" (at 58.42 26.67 0)
+    (property "Datasheet" "https://www.lcsc.com/datasheet/lcsc_datasheet_2304140030_ST-Semtech-MM1Z12_C86234.pdf" (at 58.42 26.67 0)
       (effects (font (size 1.27 1.27)) hide)
     )

Commit message: July update
Parts:
- removed D2: B5819W, Diode_SMD:D_SOD-123, symbol Device:D_Schottky
- removed U3: LM2842X, Package_TO_SOT_SMD:TSOT-23-6, symbol Regulator_Switching:LM2842X
- removed U4: AP2112K-3.3, Package_TO_SOT_SMD:SOT-23-5, symbol Regulator_Linear:AP2112K-3.3
- added C8: 100nF, Capacitor_SMD:C_0402_1005Metric, symbol Device:C
- added U3: AP63203WU, Package_TO_SOT_SMD:TSOT-23-6, symbol Regulator_Switching:AP63203WU
- C19: value 220nF -> 1uF; LCSC C16772 -> C52923
- C2, C22: value 10uF -> 22uF; LCSC C15850 -> C45783
- C3: value 10uF -> 1uF; footprint Capacitor_SMD:C_0805_2012Metric -> Capacitor_SMD:C_0402_1005Metric; LCSC C15850 -> C52923
- L1: value 10uH -> 4.7uH; LCSC C83442 -> C60117
- R10: value 10k -> 4.7k; LCSC C25744 -> C25900
- R11, R12: value 54.9k -> 33k; LCSC C11626 -> C25779
- R13, R16: value 54.9k -> 4.7k; LCSC C11626 -> C25900
- R8: value 10k -> 33k; LCSC C25744 -> C25779
Connections:
- net +3V3: now also C2.2, C22.2, D1.2 (A), L1.2, R8.1, U3.1 (FB); no longer C2.1, R16.1
- net +5V: no longer C22.2, C3.2, D1.2 (A), L1.2, R11.1
- net ADDR_0: now also JP3.2 (B), U5.35 (GPIO23); no longer U5.15 (GPIO12)
- net ADDR_1: now also JP4.2 (B), U5.34 (GPIO22); no longer U5.16 (GPIO13)
- net GND: now also C19.2, C2.1, C3.2, R11.2, U3.4 (GND); no longer C2.2, C3.1, R13.2, R8.2
- net M1_SENSE: now also C19.1, R16.2; no longer R14.1, U1.6 (IPROPI)
- net M2_SENSE: now also C3.1, R13.2; no longer R17.1, U2.6 (IPROPI)
- net TX_BUFFERED: now also R8.2; no longer R16.2
- net VCC: now also U3.2 (EN), U3.3 (IN)
- net VREF: now also R11.1; no longer R13.1
- net at L1.1: now also C8.2, U3.5 (SW); no longer C19.2
- net ADDR_2: no longer names the net of U5.17 (GPIO14)
- new net: R13.1, R17.1, U2.6 (IPROPI)
- new net: R14.1, R16.1, U1.6 (IPROPI)
- new net: C8.1, U3.6 (BST)
Other:
- moved on the sheet: L1
