File: hardware/motor-driver/motor-driver.kicad_pcb (KiCad board)
At the start: 4 copper layers, 60 x 50 mm, 27 parts, among them J1 Screw_Terminal_01x02, J10 Conn_01x02, J11 Conn_01x02, J12 Conn_01x02, J2 Screw_Terminal_01x02, J3 Screw_Terminal_01x02, J4 Conn_01x06, J5 Conn_01x06, J6 Conn_01x04, J7 Conn_01x04, J8 Conn_01x04, J9 Conn_01x04, Q1 AO4407A, U1 TLE9201SG, U2 TLE9201SG, U3 RP2040-castaway

Commit message: Initial commit for  version 2
Parts:
- added C10: 100nF, Capacitor_SMD:C_0402_1005Metric, F.Cu at (148.9, 113.2)
- added C11: 100nF, Capacitor_SMD:C_0402_1005Metric, F.Cu at (149.9, 113.2)
- added C12: 100nF, Capacitor_SMD:C_0402_1005Metric, F.Cu at (143.9, 117.7)
- added C13: 100nF, Capacitor_SMD:C_0402_1005Metric, F.Cu at (144.3, 121.4)
- added C14: 100nF, Capacitor_SMD:C_0402_1005Metric, F.Cu at (144.7, 124.3)
- added C15: 100nF, Capacitor_SMD:C_0402_1005Metric, F.Cu at (155.0, 117.5)
- added C16: 100nF, Capacitor_SMD:C_0402_1005Metric, F.Cu at (155.0, 121.7)
- added C17: 100nF, Capacitor_SMD:C_0402_1005Metric, F.Cu at (149.7, 125.5)
- added C18: 100nF, Capacitor_SMD:C_0402_1005Metric, F.Cu at (152.5, 128.0)
- added C19: 220nF, Capacitor_SMD:C_0402_1005Metric, F.Cu at (143.9, 114.9)
- added C2: 10uF, Capacitor_SMD:C_0805_2012Metric, F.Cu at (141.5, 131.3)
- added C20: 30pF, Capacitor_SMD:C_0402_1005Metric, F.Cu at (151.1, 110.0)
- added C21: 30pF, Capacitor_SMD:C_0402_1005Metric, F.Cu at (156.3, 111.3)
- added C22: 10uF, Capacitor_SMD:C_0805_2012Metric, F.Cu at (139.9, 110.4)
- added C23: 100nF, Capacitor_SMD:C_0402_1005Metric, F.Cu at (162.6, 115.3)
- added C3: 10uF, Capacitor_SMD:C_0805_2012Metric, F.Cu at (141.5, 124.0)
- added C4: 10uF, Capacitor_SMD:C_1206_3216Metric, F.Cu at (146.7, 108.6)
- added C5: 1uF, Capacitor_SMD:C_0402_1005Metric, F.Cu at (146.7, 124.3)
- added C6: 1uF, Capacitor_SMD:C_0402_1005Metric, F.Cu at (145.7, 124.3)
- added C9: 100nF, Capacitor_SMD:C_0402_1005Metric, F.Cu at (150.8, 125.5)
- added D2: B5819W, Diode_SMD:D_SOD-123, F.Cu at (142.9, 109.1)
- added D3: WS2812B-mini, LED_SMD:LED_SK6812MINI_PLCC4_3.5x3.5mm_P1.75mm, F.Cu at (139.1, 119.3)
- added D4: WS2812B-mini, LED_SMD:LED_SK6812MINI_PLCC4_3.5x3.5mm_P1.75mm, F.Cu at (161.2, 118.9)
- added D5: MM1Z12, Diode_SMD:D_SOD-123, F.Cu at (160.4, 106.6)
- added D6: SMF22CA, Diode_SMD:D_SOD-123F, F.Cu at (152.0, 99.4)
- added G***: LOGO, Shurik:my_logo, B.Cu at (150.0, 125.0)
- added J13: Conn_01x01, Connector_PinHeader_2.54mm:PinHeader_1x01_P2.54mm_Vertical, F.Cu at (160.3, 133.1)
- added J14: USB_B_Micro, shurik-personal:USB_Micro-B_Amphenol_10118194_Horizontal, F.Cu at (150.0, 132.3)
- added JP3: SolderJumper_2_Open, Jumper:SolderJumper-2_P1.3mm_Open_TrianglePad1.0x1.5mm, B.Cu at (154.7, 110.9)
- added L1: 10uH, Inductor_SMD:L_Taiyo-Yuden_NR-40xx, F.Cu at (141.1, 113.9)
- added R10: 10k, Resistor_SMD:R_0402_1005Metric, F.Cu at (138.2, 127.8)
- added R11: 54.9k, Resistor_SMD:R_0402_1005Metric, F.Cu at (149.7, 111.1)
- added R12: 54.9k, Resistor_SMD:R_0402_1005Metric, F.Cu at (163.3, 106.6)
- added R2: 1k, Resistor_SMD:R_0402_1005Metric, F.Cu at (160.2, 129.7)
- added R3: 10K, Resistor_SMD:R_0402_1005Metric, F.Cu at (157.6, 129.7)
- added R4: 1k, Resistor_SMD:R_0402_1005Metric, F.Cu at (151.1, 112.3)
- added R5: 27, Resistor_SMD:R_0402_1005Metric, F.Cu at (148.7, 124.3)
- added R6: 27, Resistor_SMD:R_0402_1005Metric, F.Cu at (147.7, 124.3)
- added R7: 10k, Resistor_SMD:R_0402_1005Metric, F.Cu at (158.6, 113.4)
- added R8: 10k, Resistor_SMD:R_0402_1005Metric, F.Cu at (148.7, 111.1)
- added R9: 10k, Resistor_SMD:R_0402_1005Metric, F.Cu at (138.2, 129.2)
- added SW1: SW_Push, Button_Switch_SMD:SW_SPST_PTS810, F.Cu at (159.9, 110.9)
- added U4: AP2120N-3.3, Package_TO_SOT_SMD:SOT-23, F.Cu at (141.5, 127.6)
- added U5: RP2040, RP2040_minimal:RP2040-QFN-56, F.Cu at (149.7, 118.7)
- added U6: W25Q16JVS, Package_SO:SOIC-8_5.23x5.23mm_P1.27mm, F.Cu at (158.4, 126.1)
- added Y1: X322512MSB4SI, Crystal:Crystal_SMD_Abracon_ABM8G-4Pin_3.2x2.5mm, F.Cu at (153.7, 111.5)
- C7: renamed from C2; footprint Capacitor_SMD:C_0805_2012Metric -> Capacitor_SMD:C_0402_1005Metric
- C8: renamed from C3; footprint Capacitor_SMD:C_0805_2012Metric -> Capacitor_SMD:C_0402_1005Metric
- D1: footprint LED_SMD:LED_0805_2012Metric -> LED_SMD:LED_0603_1608Metric
- J1, J2, J3: footprint TerminalBlock_Phoenix:TerminalBlock_Phoenix_MKDS-1,5-2_1x02_P5.00mm_Horizontal -> shurik-personal:TerminalBlock_Phoenix_MKDS-1,5-2_1x02_P5.00mm_Horizontal_nosilk
- J10, J11: footprint shurik-personal:JST_VH_S2P-VH_1x02_P3.96mm_Horizontal -> Shurik:JST_VH_B2P-VH-B_1x02_P3.96mm_Vertical-nosilk
- J12: footprint shurik-personal:JST_VH_S2P-VH_1x02_P3.96mm_Horizontal -> Connector_AMASS:AMASS_XT30UPB-M_1x02_P5.0mm_Vertical
- Q1: value AO4407A -> AO4407C
- R1: value 2K -> 3.3k; footprint Resistor_SMD:R_0805_2012Metric -> Resistor_SMD:R_0402_1005Metric
- U3: value RP2040-castaway -> LM2842X; footprint shurik-personal:RP2040-castaway -> Package_TO_SOT_SMD:TSOT-23-6
- moved D1 27.7 mm to (138.7, 124.1)
- moved R1 27.5 mm to (138.2, 126.4), turned to 0 degrees
- moved U3 11.2 mm to (145.9, 111.9), turned to 90 degrees
- moved JP2 9.48 mm to (152.2, 110.9), turned to 90 degrees
- moved J11 5.66 mm to (164.5, 90.0), turned to 0 degrees
- moved JP1 5.53 mm to (149.6, 110.9), turned to 90 degrees
- moved J10 5.48 mm to (131.8, 90.0), turned to 0 degrees
- moved C1 4.14 mm to (153.6, 106.7)
- moved J12 4.03 mm to (152.5, 90.0)
- moved J1 3.00 mm to (136.0, 93.0)
- moved J2 3.00 mm to (169.0, 93.0)
- moved J3 3.00 mm to (152.5, 93.0)
- moved Q1 1.20 mm to (146.4, 102.0)
- moved C7 0.81 mm to (137.6, 110.8)
Connections:
- D1 pad 2: VCC -> +5V
- J10 pad 1: /M1A -> /M1B
- J10 pad 2: /M1B -> /M1A
- J11 pad 1: /M2A -> /M2B
- J11 pad 2: /M2B -> /M2A
- J6 pad 2: +3V3 -> unconnected-(J6-Pad2)
- J7 pad 2: +3V3 -> unconnected-(J7-Pad2)
- JP1 pad 1: Net-(JP1-Pad1) -> /ADDR_0
- JP2 pad 1: Net-(JP2-Pad1) -> /ADDR_1
- Q1 pad 4: GND -> Net-(Q1-Pad4)
- U1 pad 11: /ENABLE -> /M1_ENABLE
- U2 pad 11: /ENABLE -> /M2_ENABLE
- U3 pad 1: /SDA -> Net-(C19-Pad1)
- U3 pad 2: /SCL -> GND
- U3 pad 3: /M2_DIR -> Net-(R11-Pad2)
- U3 pad 4: /M2_PWM -> VCC
- U3 pad 5: Net-(JP2-Pad1) -> VCC
- U3 pad 6: Net-(JP1-Pad1) -> Net-(C19-Pad2)
Routing:
- net GND: track 26.6 -> 91.2 mm, vias 10 -> 60
- net /ENABLE: track 49.2 -> 0.00 mm, vias 2 -> 0
- net +5V: track 0.00 -> 47.6 mm, vias 0 -> 3
- net +3V3: track 83.6 -> 121.7 mm, vias 5 -> 12
- net /M1_ENABLE: track 0.00 -> 27.9 mm, vias 0 -> 2
- net Net-(D3-Pad4): track 0.00 -> 25.2 mm, vias 0 -> 2
- net /QSPI_SS: track 0.00 -> 21.7 mm
- net +1V1: track 0.00 -> 20.5 mm, vias 0 -> 2
- net /RUN: track 0.00 -> 18.5 mm, vias 0 -> 2
- net /QSPI_SD1: track 0.00 -> 16.3 mm
- net Net-(Q1-Pad4): track 0.00 -> 16.1 mm
- net /M2_ENABLE: track 0.00 -> 16.0 mm
- net /SDA: track 36.7 -> 50.6 mm, vias 0 -> 2
- net /SCL: track 37.6 -> 51.0 mm, vias 0 -> 2
- net /QSPI_SD2: track 0.00 -> 12.2 mm
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- added copper zone on F.Cu, net +3V3
- added copper zone on In1.Cu, net GND
Other:
- board text added: "0"
- board text added: "1"
- board text added: "2"
- board text added: "BOOTSEL"
- board text added: "Heatsink area"
- board text added: "JLCJLCJLCJLC"
- board text added: "Personal Robotics Motor Controller motor-controller.rtfd.io"
- board text added: "RESET"
- board text added: "v 2.0, Feb 2022"
- board text removed: "BIT0"
- board text removed: "BIT1"
- board text removed: "Personal Robotics Motor Controller"
- board text removed: "RP2040 CastAway"

Commit message: starting work on v3
Parts:
- removed C23, C8: 100nF, Capacitor_SMD:C_0402_1005Metric
- removed D4: WS2812B-mini, LED_SMD:LED_SK6812MINI_PLCC4_3.5x3.5mm_P1.75mm
- added C24: 22nF, Capacitor_SMD:C_0402_1005Metric, F.Cu at (126.1, 110.0)
- added C25: 100nF, Capacitor_SMD:C_0402_1005Metric, F.Cu at (126.1, 108.0)
- added C26: 22nF, Capacitor_SMD:C_0402_1005Metric, F.Cu at (163.5, 110.9)
- added JP4: SolderJumper_2_Open, Jumper:SolderJumper-2_P1.3mm_Open_TrianglePad1.0x1.5mm, B.Cu at (142.5, 122.1)
- added R13: 54.9k, Resistor_SMD:R_0402_1005Metric, F.Cu at (140.6, 108.2)
- added R14: 1.5k, Resistor_SMD:R_0402_1005Metric, F.Cu at (136.1, 107.0)
- added R15: 10k, Resistor_SMD:R_0402_1005Metric, F.Cu at (175.0, 108.8)
- added R16: 54.9k, Resistor_SMD:R_0402_1005Metric, F.Cu at (164.5, 128.5)
- added R17: 1.5k, Resistor_SMD:R_0402_1005Metric, F.Cu at (175.8, 106.3)
- added U7: 74LVC1G126, Package_TO_SOT_SMD:SOT-23-5, F.Cu at (161.6, 121.0)
- D1: footprint LED_SMD:LED_0603_1608Metric -> LED_SMD:LED_0805_2012Metric
- D3: value WS2812B-mini -> SK6812MINI
- J6, J7: footprint Connector_JST:JST_SH_SM04B-SRSS-TB_1x04-1MP_P1.00mm_Horizontal -> Connector_JST:JST_PH_B4B-PH-K_1x04_P2.00mm_Vertical
- U1, U2: value TLE9201SG -> DRV8874PWPR; footprint Package_SO:Infineon_PG-DSO-12-11_ThermalVias -> shurik-personal:HTSSOP-16-1EP_4.4x5mm_P0.65mm_EP3.4x5mm_Mask2.46x3.55mm_ThermalVias_reduced
- U4: value AP2120N-3.3 -> AP2112K-3.3; footprint Package_TO_SOT_SMD:SOT-23 -> Package_TO_SOT_SMD:SOT-23-5
- moved C7 25.9 mm to (163.4, 109.6), turned to 0 degrees
- moved JP2 23.4 mm to (167.5, 128.5)
- moved JP1 23.1 mm to (134.5, 128.3)
- moved D3 21.7 mm to (160.6, 116.8), turned to 180 degrees
- moved R9 20.3 mm to (136.8, 108.9)
- moved R10 19.6 mm to (139.0, 108.2), turned to 90 degrees
- moved JP3 18.8 mm to (139.6, 122.1)
- moved R12 4.39 mm to (159.4, 104.6), turned to 180 degrees
- moved J6 3.54 mm to (163.5, 131.5)
- moved J13 2.83 mm to (157.5, 133.4)
- moved J7 2.55 mm to (130.5, 131.5)
- moved C15 1.26 mm to (155.4, 116.3), turned to 90 degrees
- moved U1 1.12 mm to (131.0, 108.5)
- moved U2 1.12 mm to (169.0, 108.5)
- moved R2 0.96 mm to (159.2, 129.6)
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Connections:
- C7 pad 2: GND -> Net-(U2-VCP)
- D3 pad 1: +3V3 -> unconnected-(D3-DOUT-Pad1)
- D3 pad 2: unconnected-(D3-Pad2) -> GND
- D3 pad 3: GND -> /NEOPIXEL
- D3 pad 4: Net-(D3-Pad4) -> +3V3
- J6 pad 1: GND -> /TX_BUFFERED
- J6 pad 2: unconnected-(J6-Pad2) -> /RX
- J6 pad 3: /SDA -> Net-(J6-Pin_3)
- J6 pad 4: /SCL -> GND
- J7 pad 1: GND -> /TX_BUFFERED
- J7 pad 2: unconnected-(J7-Pad2) -> /RX
- J7 pad 3: /SDA -> Net-(J7-Pin_3)
- J7 pad 4: /SCL -> GND
- JP1 pad 1: /ADDR_0 -> Net-(J7-Pin_3)
- JP1 pad 2: GND -> +3V3
- JP2 pad 1: /ADDR_1 -> Net-(J6-Pin_3)
- JP2 pad 2: GND -> +3V3
- JP3 pad 1: /ADDR_2 -> GND
- JP3 pad 2: GND -> Net-(JP3-B)
- R10 pad 2: /SDA -> /VREF
- R9 pad 2: /SCL -> /M1_FLAG
- U1 pad 1: /M1_DIR -> /M1_PWM
- U1 pad 10: GND -> /M1B
- U1 pad 11: /M1_ENABLE -> VCC
- U1 pad 12: /M1_PWM -> Net-(U1-VCP)
- U1 pad 13: GND -> Net-(U1-CPH)
- U1 pad 2: +3V3 -> /M1_DIR
- U1 pad 3: /M1_FLAG -> /M1_ENABLE
- U1 pad 4: VCC -> /M1_FLAG
- U1 pad 5: /M1A -> /VREF
- U1 pad 6: GND -> /M1_SENSE
- U1 pad 7: /M1B -> GND
- U1 pad 8: GND -> /M1A
- U2 pad 1: /M2_DIR -> /M2_PWM
- U2 pad 10: GND -> /M2B
- U2 pad 11: /M2_ENABLE -> VCC
- U2 pad 12: /M2_PWM -> Net-(U2-VCP)
- U2 pad 13: GND -> Net-(U2-CPH)
- U2 pad 2: +3V3 -> /M2_DIR
- U2 pad 3: /M2_FLAG -> /M2_ENABLE
- U2 pad 4: VCC -> /M2_FLAG
- U2 pad 5: /M2A -> /VREF
- U2 pad 6: GND -> /M2_SENSE
- U2 pad 7: /M2B -> GND
- U2 pad 8: GND -> /M2A
- U4 pad 1: GND -> +5V
- U4 pad 2: +3V3 -> GND
- U5 pad 2: /SDA -> /TX
- U5 pad 3: /SCL -> /RX
- U5 pad 31: /M1_DIR -> /M1_FLAG
- U5 pad 36: /M1_FLAG -> Net-(JP4-B)
- U5 pad 37: unconnected-(U5-Pad37) -> Net-(JP3-B)
- U5 pad 38: unconnected-(U5-Pad38) -> /M1_ENABLE
- U5 pad 39: /M1_ENABLE -> /M1_DIR
- U5 pad 4: /M2_DIR -> /TX_CTRL
- U5 pad 5: /NEOPIXEL -> /M2_FLAG
- U5 pad 6: unconnected-(U5-Pad6) -> /NEOPIXEL
- U5 pad 7: /M2_FLAG -> /M2_DIR
Routing:
- net /RX: track 0.00 -> 55.8 mm, vias 0 -> 1
- net /VREF: track 0.00 -> 55.5 mm, vias 0 -> 2
- net /SCL: track 51.0 -> 0.00 mm, vias 2 -> 0
- net /SDA: track 50.6 -> 0.00 mm, vias 2 -> 0
- net /TX_BUFFERED: track 0.00 -> 44.2 mm
- net Net-(D3-Pad4): track 25.2 -> 0.00 mm, vias 2 -> 0
- net /M2B: track 3.21 -> 15.0 mm
- net /M2_PWM: track 14.8 -> 26.1 mm, vias 0 -> 2
- net /ENC2_B: track 47.3 -> 37.3 mm
- net Net-(JP3-B): track 0.00 -> 9.24 mm, vias 0 -> 1
- net /M1_PWM: track 28.0 -> 19.0 mm, vias 2 -> 0
- net /M2_ENABLE: track 16.0 -> 24.7 mm, vias 0 -> 2
- net /M1_ENABLE: track 27.9 -> 19.2 mm, vias 2 -> 0
- net /M2_FLAG: track 28.4 -> 36.9 mm
- net /M1A: track 6.66 -> 14.5 mm
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- added copper zone on In2.Cu, net +3V3
- added copper zone on In2.Cu, net VCC
- removed copper zone on In1.Cu, net +3V3
- removed copper zone on In1.Cu, net VCC
Other:
- board text added: "3V3"
- board text added: "ID0"
- board text added: "ID1"
- board text added: "RX"
- board text added: "TX"
- board text added: "UART"
- board text added: "v 3.0, July 2024"
- board text removed: "0"
- board text removed: "1"
- board text removed: "2"
- board text removed: "I2C"
- board text removed: "I2C ADDR"
- board text removed: "v 2.0, Feb 2022"

Commit message: version 3.0.0-beta1
Parts:
- L1: footprint Inductor_SMD:L_Taiyo-Yuden_NR-40xx -> Inductor_SMD:L_Sunlord_SWPA4018S
- moved C13 0.79 mm to (144.3, 122.2)
Connections:
- U5 pad 34: unconnected-(U5-GPIO22-Pad34) -> Net-(JP4-B)
- U5 pad 35: unconnected-(U5-GPIO23-Pad35) -> Net-(JP3-B)
- U5 pad 36: Net-(JP4-B) -> /M1_ENABLE
- U5 pad 37: Net-(JP3-B) -> /M1_DIR
- U5 pad 38: /M1_ENABLE -> /M1_PWM
- U5 pad 39: /M1_DIR -> /M1_SENSE
- U5 pad 40: /M1_PWM -> /M2_SENSE
Routing:
- net /M2_SENSE: track 4.99 -> 52.5 mm, vias 0 -> 3
- net /M1_SENSE: track 3.27 -> 25.0 mm, vias 0 -> 2
- net +1V1: track 15.7 -> 20.5 mm, vias 0 -> 2
- net +3V3: track 121.9 -> 117.9 mm, vias 13 -> 14
- net /ENC1_A: track 34.4 -> 36.6 mm
- net /VREF: track 55.5 -> 56.3 mm

Commit message: July update
Parts:
- removed D2: B5819W, Diode_SMD:D_SOD-123
- removed U4: AP2112K-3.3, Package_TO_SOT_SMD:SOT-23-5
- added C8: 100nF, Capacitor_SMD:C_0402_1005Metric, F.Cu at (144.5, 114.7)
- C19: value 220nF -> 1uF
- C2, C22: value 10uF -> 22uF
- C3: value 10uF -> 1uF; footprint Capacitor_SMD:C_0805_2012Metric -> Capacitor_SMD:C_0402_1005Metric
- L1: value 10uH -> 4.7uH
- R10: value 10k -> 4.7k
- R11, R12: value 54.9k -> 33k
- R13, R16: value 54.9k -> 4.7k
- R8: value 10k -> 33k
- U3: value LM2842X -> AP63203WU
- moved R16 26.7 mm to (139.1, 120.3), turned to 0 degrees
- moved C2 23.5 mm to (141.5, 107.8)
- moved R8 23.5 mm to (164.5, 128.5), turned to 180 degrees
- moved C3 15.7 mm to (149.6, 110.5), turned to 0 degrees
- moved R11 10.00 mm to (141.1, 106.1), turned to 0 degrees
- moved R13 9.43 mm to (149.4, 111.6), turned to 0 degrees
- moved C19 8.06 mm to (139.1, 121.4), turned to 180 degrees
- moved R1 3.72 mm to (141.9, 126.2), turned to 180 degrees
- moved D1 3.44 mm to (141.8, 123.5)
- moved R10 1.61 mm to (139.2, 106.6)
- moved C22 1.56 mm to (141.4, 109.9)
- moved C4 1.04 mm to (146.2, 109.5)
- moved R15 0.70 mm to (175.7, 108.8)
- moved L1 0.62 mm to (141.2, 113.3)
- moved U3 0.61 mm to (145.6, 112.4), turned to 180 degrees
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Connections:
- C19 pad 1: Net-(U3-BOOST) -> /M1_SENSE
- C19 pad 2: Net-(D2-K) -> GND
- C2 pad 1: +3V3 -> GND
- C2 pad 2: GND -> +3V3
- C22 pad 2: +5V -> +3V3
- C3 pad 1: GND -> /M2_SENSE
- C3 pad 2: +5V -> GND
- D1 pad 2: +5V -> +3V3
- JP3 pad 2: Net-(JP3-B) -> /ADDR_0
- JP4 pad 2: Net-(JP4-B) -> /ADDR_1
- L1 pad 1: Net-(D2-K) -> Net-(U3-SW)
- L1 pad 2: +5V -> +3V3
- R11 pad 1: +5V -> /VREF
- R11 pad 2: Net-(U3-FB) -> GND
- R13 pad 1: /VREF -> Net-(U2-IPROPI)
- R13 pad 2: GND -> /M2_SENSE
- R14 pad 1: /M1_SENSE -> Net-(U1-IPROPI)
- R16 pad 1: +3V3 -> Net-(U1-IPROPI)
- R16 pad 2: /TX_BUFFERED -> /M1_SENSE
- R17 pad 1: /M2_SENSE -> Net-(U2-IPROPI)
- R8 pad 1: Net-(U3-FB) -> +3V3
- R8 pad 2: GND -> /TX_BUFFERED
- U1 pad 6: /M1_SENSE -> Net-(U1-IPROPI)
- U2 pad 6: /M2_SENSE -> Net-(U2-IPROPI)
- U3 pad 1: Net-(U3-BOOST) -> +3V3
- U3 pad 2: GND -> VCC
- U3 pad 3: Net-(U3-FB) -> VCC
- U3 pad 4: VCC -> GND
- U3 pad 5: VCC -> Net-(U3-SW)
- U3 pad 6: Net-(D2-K) -> Net-(U3-BST)
- U5 pad 15: /ADDR_0 -> unconnected-(U5-GPIO12-Pad15)
- U5 pad 16: /ADDR_1 -> unconnected-(U5-GPIO13-Pad16)
- U5 pad 17: /ADDR_2 -> unconnected-(U5-GPIO14-Pad17)
- U5 pad 34: Net-(JP4-B) -> /ADDR_1
- U5 pad 35: Net-(JP3-B) -> /ADDR_0
Routing:
- net +5V: track 43.2 -> 0.00 mm, vias 3 -> 0
- net VCC: track 6.47 -> 45.2 mm
- net Net-(U2-IPROPI): track 0.00 -> 37.8 mm, vias 0 -> 2
- net /M2_SENSE: track 52.5 -> 17.0 mm, vias 3 -> 2
- net Net-(U1-IPROPI): track 0.00 -> 17.7 mm, vias 0 -> 2
- net /M1_SENSE: track 25.0 -> 8.32 mm, vias 2 -> 0
- net /M2_DIR: track 30.7 -> 42.5 mm
- net /M2_PWM: track 26.1 -> 35.9 mm
- net GND: track 98.1 -> 88.9 mm, vias 58 -> 60
- net /ADDR_0: track 0.00 -> 9.09 mm, vias 0 -> 1
- net Net-(JP3-B): track 9.08 -> 0.00 mm, vias 1 -> 0
- net /M2_ENABLE: track 24.7 -> 33.7 mm
- net Net-(D2-K): track 7.32 -> 0.00 mm
- net /ADDR_1: track 0.00 -> 6.24 mm, vias 0 -> 1
- net Net-(JP4-B): track 6.23 -> 0.00 mm, vias 1 -> 0
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- added copper zone on B.Cu, net VCC
